File: DAC_filters.kicad_sch (KiCad schematic)
At the start: 24 parts

Commit message: finished individual block placement and started integrating, might need to change the AFEs length
Parts:
- C901, C905, C909, C910: footprint (none) -> Capacitor_SMD:C_0603_1608Metric; MPN (none) -> CGA0603X7R122K500JT
- C902, C906, C911, C912: footprint (none) -> Capacitor_SMD:C_0603_1608Metric; MPN (none) -> FCC0603B471K500CT
- C903, C904, C907, C908: value 1.1nF -> 1.2nF; footprint (none) -> Capacitor_SMD:C_0603_1608Metric; MPN (none) -> CGA0603X7R122K500JT
- L901, L903, L905, L906: footprint (none) -> Inductor_SMD:L_0603_1608Metric; MPN (none) -> WI0603LD470KST-HF
- L902, L904, L907, L908: footprint (none) -> Inductor_SMD:L_0805_2012Metric; MPN (none) -> MLI2012F-390KT
- R404, R901, R902, R903: footprint (none) -> Resistor_SMD:R_0603_1608Metric; MPN (none) -> PTFR0603B200RP9
Connections:
- net DAC_OUT1: now also C908.1; no longer C903.1
- net DAC_OUT2: now also C907.1; no longer C904.1
- net DAC_OUT3: now also C904.1; no longer C907.1
- net DAC_OUT4: now also C903.1; no longer C908.1
