File: NadyScope.kicad_pcb (KiCad board)
At the start: 2 copper layers, 124 parts, among them IC301 TLA2518IRTER, J201 Debugging Connector, J301 ADC AFE IN 1, J302 ADC AFE IN 2, J401 DAC OUT, J402 DAC Output 2, J403 DAC Output 3, J405 MCU DAC OUT, J406 DAC Output 1, J407 DAC Output 5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

Commit message: DONE, ready for ordering
Parts:
- Analog Input 1: renamed from J301
- Analog Input 2: renamed from J302
- Analog Output 1: renamed from J405
- Analog Output 2: renamed from J401
- C701, C702, D301, R302, R303: moved to B.Cu
- moved J501 187.0 mm to (278.0, 122.0), turned to 0 degrees
- moved R501 182.8 mm to (275.3, 124.0), turned to -90 degrees
- moved R502 182.2 mm to (275.3, 127.3), turned to 90 degrees
- moved C502 179.5 mm to (273.7, 129.7), turned to 180 degrees
- moved U501 175.9 mm to (270.6, 125.6), turned to -90 degrees
- moved C501 173.4 mm to (267.6, 122.1)
- moved C702 29.4 mm to (218.4, 110.7)
- moved R303 27.4 mm to (218.4, 109.2)
- moved R309 26.3 mm to (227.1, 106.7), turned to 90 degrees
- moved R302 25.6 mm to (218.4, 107.6)
- moved C701 24.1 mm to (218.4, 106.1)
- moved Analog Output 1 23.7 mm to (252.6, 151.8)
- moved Q301 21.4 mm to (226.0, 103.4), turned to 180 degrees
- moved D201 21.3 mm to (241.1, 104.7), turned to 0 degrees
- moved D301 19.0 mm to (218.4, 103.9)
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Connections:
- R202 pad 1: /ADC/MCU_ADC -> /MCU/MCU_LED
- R204 pad 1: Net-(U201-IO6) -> /MCU/MCU_LED
- R401 pad 2: /DAC/DAC_SDA -> /DAC/DAC_SCL
- R402 pad 2: /DAC/DAC_SCL -> /DAC/DAC_SDA
- U201 pad 12: /ADC/ADC_SDO -> /ADC/MCU_ADC
- U201 pad 13: /ADC/ADC_SDI -> /ADC/ADC_SCLK
- U201 pad 16: /DAC/DAC_LDAC -> /ADC/ADC_SDO
- U201 pad 20: Net-(U201-IO6) -> /DAC/DAC_LDAC
- U201 pad 21: /DAC/DAC_SCL -> /DAC/DAC_SDA
- U201 pad 22: /DAC/DAC_SDA -> /DAC/DAC_SCL
- U201 pad 26: /MCU/USB_P -> /MCU/USB_N
- U201 pad 27: /MCU/USB_N -> /MCU/USB_P
- U201 pad 5: /ADC/MCU_ADC -> /MCU/MCU_LED
- U201 pad 6: /ADC/ADC_SCLK -> /ADC/ADC_SDI
- U601 pad 1: /MCU/USB_N -> /MCU/USB_P
- U601 pad 3: /MCU/USB_P -> /MCU/USB_N
- U601 pad 4: /MCU/USB_P -> /MCU/USB_N
- U601 pad 6: /MCU/USB_N -> /MCU/USB_P
Routing:
- net USB_VDD: track 0.00 -> 91.2 mm, vias 0 -> 6
- net MCU_3V3: track 0.00 -> 41.5 mm, vias 0 -> 14
- net /ADC/14dB_EN: track 0.00 -> 37.1 mm, vias 0 -> 2
- net /DAC/DAC Filters/DAC_OUT_FILT1: track 0.00 -> 23.1 mm
- net /ADC/AFE_OUT2: track 0.00 -> 22.4 mm
- net /ADC/ADC_SDI: track 0.00 -> 22.1 mm, vias 0 -> 2
- net /DAC/DAC_SDA: track 0.00 -> 21.5 mm, vias 0 -> 2
- net /DAC/DAC_SCL: track 0.00 -> 20.4 mm, vias 0 -> 2
- net /ADC/MCU_ADC: track 0.00 -> 20.3 mm
- net /DAC/DAC Filters/DAC_OUT_FILT4: track 0.00 -> 18.9 mm
- net ISO_VCC_I2C: track 0.00 -> 18.3 mm
- net /DAC/DAC_MCU: track 0.00 -> 17.6 mm
- net /ADC/ADC_CSn: track 0.00 -> 17.0 mm
- net /ADC/ADC_SDO: track 0.00 -> 15.4 mm
- net /MCU/USB_P: track 0.00 -> 14.3 mm
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- added copper zone on F.Cu, net /ADC/Attenuators/4dB_OUT
- added copper zone on B.Cu, net AVDD
- added copper zone on F.Cu, net AVDD
- added copper zone on B.Cu, net GND
- added copper zone on In1.Cu, net GND
- added copper zone on In2.Cu, net GND
- added copper zone on B.Cu, net ISO_GND_I2C
- added copper zone on F.Cu, net ISO_GND_I2C
- added copper zone on In1.Cu, net ISO_GND_I2C
- added copper zone on In2.Cu, net ISO_GND_I2C
- added copper zone on B.Cu, net MCU_3V3
- added copper zone on F.Cu, net MCU_3V3
- added copper zone on F.Cu, net Net-(U803-+)
- added copper zone on B.Cu, net USB_VDD
Other:
- board outline added: 80 x 55.2 mm
- copper layers 2 -> 4
- board text added: "Designed By: Yusuf Elnady"
- board text added: "From Signal to Certainty"
- board text added: "GND - TX - RX - 5V"
- board text added: "NadyScope"
- board text added: "VDD SDA SCL GND"
